File: RoboticsTeam-main/RoboticsPCBS/DriverBoard/DriverBoard.kicad_pcb (KiCad board)
At the start: 4 copper layers, 185 x 115 mm, 43 parts, among them J1 B4B-XH-A(LF)(SN), J10 B8B-XH-ALFSN, J11 B8B-XH-ALFSN, J12 B8B-XH-ALFSN, J13 B8B-XH-ALFSN, J14 B6B-XH-ALFSN, J15 B8B-XH-ALFSN, J16 USB_B_Micro, J17 Conn_01x02_Male, J18 Conn_01x02_Male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

Commit message: Add files via upload
Parts:
- removed the ? at (122.0, 83.4)
- removed the ? at (44.8, 148.9)
- added ?: , , F.Cu at (199.9, 78.4)
- added ?: , , F.Cu at (46.0, 147.9)
- added C7: 0.1µF, DriverBoard:0603Footprint, F.Cu at (87.4, 57.6)
- added C8: 0.1µF, DriverBoard:0603Footprint, F.Cu at (87.4, 64.4)
- added J24: B4B-XH-A(LF)(SN), DriverBoard:JST4Way, F.Cu at (169.6, 54.8)
- added J25: B4B-XH-A(LF)(SN), DriverBoard:JST4Way, F.Cu at (185.7, 54.8)
- added J26: B4B-XH-A(LF)(SN), DriverBoard:JST4Way, F.Cu at (153.5, 141.7)
- added J27: B4B-XH-A(LF)(SN), DriverBoard:JST4Way, F.Cu at (169.6, 141.7)
- added J28: B4B-XH-A(LF)(SN), DriverBoard:JST4Way, F.Cu at (185.7, 141.8)
- added J29: B4B-XH-A(LF)(SN), DriverBoard:JST4Way, F.Cu at (153.5, 54.8)
- moved J22 157.7 mm to (98.0, 141.7), turned to 0 degrees
- moved J10 113.7 mm to (165.4, 45.0)
- moved J12 101.2 mm to (139.3, 151.2)
- moved C4 85.4 mm to (199.8, 85.8), turned to 270 degrees
- moved C6 78.8 mm to (205.9, 84.3)
- moved U5 78.1 mm to (200.0, 79.7)
- moved C3 69.0 mm to (199.8, 100.7), turned to 270 degrees
- moved U4 59.7 mm to (200.0, 93.3)
- moved C5 59.2 mm to (205.9, 97.3)
- moved J11 51.2 mm to (113.3, 151.2)
- moved J13 27.4 mm to (165.4, 151.2)
- moved J9 25.4 mm to (139.3, 45.1)
- moved R2 14.0 mm to (229.2, 48.4), turned to 180 degrees
- moved C2 10.8 mm to (199.8, 122.2), turned to 270 degrees
- moved J6 10.7 mm to (137.4, 141.7)
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Connections:
- C1 pad 1: +1V8 -> +3V3
- C5 pad 1: +1V8 -> +3V3
- C6 pad 1: +1V8 -> +3V3
- J15 pad 4: Net-(J15-Pad4) -> SPI_1_CS
- J15 pad 5: Net-(J15-Pad5) -> SPI_1_MISO
- J15 pad 6: Net-(J15-Pad6) -> SPI_1_MOSI
- J15 pad 7: Net-(J15-Pad7) -> SPI_1_SCK
- J15 pad 8: Net-(J15-Pad8) -> SPI_1_INT
- U1 pad 1: Net-(U1-Pad1) -> Steer5-Enc-Aout
- U1 pad 102: Drive2-PWMA -> Drive3-PWMA
- U1 pad 104: Net-(U1-Pad104) -> Drive2-Enc-Aout
- U1 pad 105: Net-(U1-Pad105) -> Steer1-INB2
- U1 pad 109: Net-(U1-Pad109) -> Steer1-INB1
- U1 pad 110: Net-(U1-Pad110) -> Steer1-INA2
- U1 pad 111: Net-(U1-Pad111) -> Steer1-Enc-Bout
- U1 pad 112: Net-(U1-Pad112) -> Steer1-Enc-Aout
- U1 pad 117: LED2 -> Steer2-INA1
- U1 pad 118: Net-(U1-Pad118) -> Steer2-INB2
- U1 pad 119: Net-(U1-Pad119) -> Steer2-INB1
- U1 pad 122: Net-(U1-Pad122) -> Steer2-INA2
- U1 pad 123: Net-(U1-Pad123) -> SPI_1_MOSI
- U1 pad 124: Net-(U1-Pad124) -> SPI_1_MISO
- U1 pad 125: Net-(U1-Pad125) -> SPI_1_CS
- U1 pad 126: I2C-2-INT -> SPI_1_SCK
- U1 pad 127: Net-(U1-Pad127) -> Steer6-Enc-Aout
- U1 pad 128: Net-(U1-Pad128) -> SPI_1_INT
- U1 pad 129: Net-(U1-Pad129) -> Drive4-Enc-Bout
- U1 pad 13: Net-(U1-Pad13) -> Drive3-INB1
- U1 pad 132: Net-(U1-Pad132) -> Steer3-INA1
- U1 pad 137: CAN2-STBY -> Net-(U1-Pad137)
- U1 pad 141: Net-(U1-Pad141) -> Drive3-INA1
- U1 pad 142: Net-(U1-Pad142) -> Steer3-INA2
- U1 pad 15: Net-(U1-Pad15) -> Drive2-INA1
- U1 pad 18: Net-(U1-Pad18) -> Steer2-Enc-Bout
- U1 pad 19: Net-(U1-Pad19) -> Steer2-Enc-Aout
- U1 pad 2: Net-(U1-Pad2) -> Steer3-INB2
- U1 pad 20: Steer3-PWMA -> Steer2-PWMA
- U1 pad 21: Steer3-PWMB -> Steer2-PWMB
- U1 pad 22: Net-(U1-Pad22) -> Drive5-Enc-Bout
- U1 pad 24: Net-(U1-Pad24) -> Steer4-Enc-Bout
- U1 pad 3: Net-(U1-Pad3) -> Steer3-INB1
- U1 pad 34: Net-(U1-Pad34) -> Steer3-Enc-Bout
- U1 pad 35: Drive3-PWMB -> Steer1-PWMB
- U1 pad 36: Net-(U1-Pad36) -> Drive4-Enc-Aout
- U1 pad 4: Steer1-PWMA -> Steer3-PWMA
- U1 pad 40: Net-(U1-Pad40) -> Steer3-Enc-Aout
- U1 pad 41: Drive3-PWMA -> Steer1-PWMA
- U1 pad 43: Net-(U1-Pad43) -> Steer6-Enc-Bout
- U1 pad 44: Net-(U1-Pad44) -> Drive2-INA2
- U1 pad 46: Net-(U1-Pad46) -> Steer4-Enc-Aout
- U1 pad 47: Net-(U1-Pad47) -> Drive3-Enc-Bout
- U1 pad 48: CAN3-STBY -> CAN2-STBY
- U1 pad 49: Net-(U1-Pad49) -> Drive3-INA2
- U1 pad 5: Steer1-PWMB -> Steer3-PWMB
- U1 pad 56: Net-(U1-Pad56) -> I2C-2-INT
- U1 pad 57: Net-(U1-Pad57) -> CAN1-STBY
- U1 pad 64: Net-(U1-Pad64) -> Drive3-INB2
- U1 pad 65: Net-(U1-Pad65) -> CAN3-STBY
- U1 pad 66: Net-(U1-Pad66) -> Drive2-B1
- U1 pad 67: Drive2-PWMB -> Drive3-PWMB
- U1 pad 68: Net-(U1-Pad68) -> Drive5-Enc-Aout
- U1 pad 69: Net-(U1-Pad69) -> Drive3-Enc-Aout
- U1 pad 7: Net-(U1-Pad7) -> Steer1-INA1
- U1 pad 70: Net-(U1-Pad70) -> Drive1-INB1
- U1 pad 74: Net-(U1-Pad74) -> Drive2-B2
- U1 pad 75: Net-(U1-Pad75) -> Drive1-INA1
- U1 pad 76: Net-(U1-Pad76) -> Drive1-INA2
- U1 pad 77: Net-(U1-Pad77) -> Drive2-Enc-Bout
- U1 pad 79: Net-(U1-Pad79) -> Drive6-Enc-Aout
- U1 pad 81: Steer2-PWMA -> Drive2-PWMA
- U1 pad 82: Steer2-PWMB -> Drive2-PWMB
- U1 pad 88: Net-(U1-Pad88) -> Steer5-Enc-Bout
- U1 pad 90: Net-(U1-Pad90) -> LED2
- U1 pad 91: +3V3 -> Net-(U1-Pad91)
- U1 pad 93: Net-(U1-Pad93) -> Drive6-Enc-Bout
- U1 pad 96: Net-(U1-Pad96) -> Drive1-Enc-Aout
- U1 pad 97: Net-(U1-Pad97) -> Drive1-INB2
- U1 pad 98: Net-(U1-Pad98) -> Drive1-Enc-Bout
- U2 pad 10: Net-(U2-Pad10) -> VCCIO
- U2 pad 3: Net-(U2-Pad3) -> VCCIO
- U3 pad 5: +1V8 -> +3V3
- U4 pad 5: +1V8 -> +3V3
- U5 pad 5: +1V8 -> +3V3
Routing:
- net Steer1-PWMA: track 20.2 -> 120.5 mm
- net SPI_1_MOSI: track 0.00 -> 93.0 mm
- net GND: track 76.3 -> 160.3 mm, vias 14 -> 31
- net CAN3-RXD: track 0.00 -> 69.0 mm
- net SPI_1_MISO: track 0.00 -> 67.8 mm
- net +5V: track 30.1 -> 95.8 mm, vias 1 -> 17
- net CAN2-STBY: track 0.00 -> 64.5 mm
- net CAN2-RXD: track 16.8 -> 78.8 mm
- net Net-(J20-Pad2): track 104.6 -> 43.0 mm
- net Net-(J17-Pad2): track 84.6 -> 23.0 mm
- net Drive3-PWMA: track 108.9 -> 54.0 mm
- net Steer6-Enc-Bout: track 0.00 -> 50.7 mm
- net I2C-2-INT: track 20.6 -> 67.8 mm
- net CAN3-TXD: track 20.6 -> 64.4 mm
- net CAN2-TXD: track 17.8 -> 59.9 mm
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- added copper zone on GND, net GND
Other:
- board size 185 x 115 mm -> 184.7 x 118.4 mm
- board text added: "SPI"
- board text added: "Steer 1 Enc"
- board text added: "Steer 2 Enc"
- board text added: "Steer 3 Enc"
- board text added: "Steer 4 Enc"
- board text added: "Steer 5 Enc"
- board text added: "Steer 6 Enc"

Commit message: Add files via upload
Parts:
- removed the ? at (46.0, 147.9)
- removed J22: Conn_01x02_Male, DriverBoard:2PinHeader
- added ?: , , F.Cu at (169.6, -103.5)
- added ?: , , F.Cu at (169.6, 0.00)
- added ?: , , F.Cu at (0.10, -103.5)
- added J30: B4B-XH-A(LF)(SN), DriverBoard:JST4Way, F.Cu at (96.5, 149.0)
- added REF**: M3Drill, DriverBoard:M3Drill, F.Cu at (65.0, 150.3)
- R1, R2: footprint DriverBoard:LEDResistor -> DriverBoard:0603Footprint
- moved R2 7.10 mm to (222.1, 48.4)
- moved R1 7.02 mm to (222.1, 58.9)
- moved D1 3.10 mm to (214.1, 58.8)
- moved D2 3.10 mm to (214.1, 48.5)
Connections:
- U1 pad 116: LED1 -> Net-(U1-Pad116)
- U1 pad 17: Net-(U1-Pad17) -> (no net)
- U1 pad 6: Net-(U1-Pad6) -> (no net)
- U1 pad 89: Net-(U1-Pad89) -> LED1
Routing:
- net I2C-2-INT: track 67.8 -> 41.8 mm
- net SabreTX: track 31.6 -> 43.3 mm
- net GND: track 160.3 -> 150.4 mm, vias 31 -> 30
- net LED1: track 23.1 -> 25.2 mm
- net LED2: track 28.1 -> 29.3 mm
- net Net-(D1-Pad1): track 4.09 -> 4.64 mm
Other:
- board size 184.7 x 118.4 mm -> 184.5 x 118.4 mm
