File: RoboticsPCBS/DriverBoard/DriverBoard.kicad_pcb (KiCad board)
At the start: 4 copper layers, 43 parts, among them J1 B4B-XH-A(LF)(SN), J10 B8B-XH-ALFSN, J11 B8B-XH-ALFSN, J12 B8B-XH-ALFSN, J13 B8B-XH-ALFSN, J14 B6B-XH-ALFSN, J15 B8B-XH-ALFSN, J16 USB_B_Micro, J17 Conn_01x02_Male, J18 Conn_01x02_Male, J19 B2B-XH-A(LF)(SN), J2 B4B-XH-A(LF)(SN), J20 B2B-XH-A(LF)(SN), J21 B2B-XH-A(LF)(SN), J22 Conn_01x02_Male, J23 Conn_01x02_Male, J3 B4B-XH-A(LF)(SN), J4 B4B-XH-A(LF)(SN), J5 B4B-XH-A(LF)(SN), J6 B4B-XH-A(LF)(SN), J7 B6B-XH-ALFSN, J8 B8B-XH-ALFSN, J9 B8B-XH-ALFSN, U1 STM32F767ZITx, U2 FT230XS, U3 MCP2562, U4 MCP2562, U5 MCP2562-E_SN

Commit message: Add files via upload
Parts:
- removed the ? at (134.5, 58.4)
- removed the ? at (154.3, 63.5)
- removed J16: USB_B_Micro, DriverBoard:MicroBVert
- removed J22: Conn_01x02_Male, DriverBoard:2PinHeader
- removed U2: FT230XS, DriverBoard:FT230XS
- added ?: , , F.Cu at (0.10, -103.5)
- added ?: , , F.Cu at (199.9, 78.4)
- added J24: B4B-XH-A(LF)(SN), DriverBoard:JST4Way, F.Cu at (169.6, 54.8)
- added J25: B4B-XH-A(LF)(SN), DriverBoard:JST4Way, F.Cu at (185.7, 54.8)
- added J26: B4B-XH-A(LF)(SN), DriverBoard:JST4Way, F.Cu at (153.5, 141.7)
- added J27: B4B-XH-A(LF)(SN), DriverBoard:JST4Way, F.Cu at (169.6, 141.7)
- added J28: B4B-XH-A(LF)(SN), DriverBoard:JST4Way, F.Cu at (185.7, 141.8)
- added J29: B4B-XH-A(LF)(SN), DriverBoard:JST4Way, F.Cu at (153.5, 54.8)
- added J30: B4B-XH-A(LF)(SN), DriverBoard:JST4Way, F.Cu at (96.5, 149.0)
- added REF**: M3Drill, DriverBoard:M3Drill, F.Cu at (234.5, 47.0)
- added REF**: M3Drill, DriverBoard:M3Drill, F.Cu at (234.5, 150.2)
- added REF**: M3Drill, DriverBoard:M3Drill, F.Cu at (65.0, 150.3)
- R1, R2: footprint DriverBoard:LEDResistor -> DriverBoard:0603Footprint
- U3, U4: value MCP2562 -> MCP2562-E_SN
- moved J12 121.3 mm to (139.3, 151.2)
- moved J1 107.8 mm to (105.3, 54.6)
- moved J2 106.7 mm to (105.3, 141.7)
- moved D2 99.5 mm to (214.1, 48.5)
- moved J15 98.3 mm to (220.8, 145.5)
- moved R2 96.6 mm to (222.1, 48.4)
- moved J5 92.9 mm to (137.4, 54.8)
- moved J14 91.1 mm to (204.0, 151.2), turned to 180 degrees
- moved J3 87.7 mm to (121.4, 54.8)
- moved J7 86.2 mm to (204.0, 45.0), turned to 180 degrees
- moved D1 79.1 mm to (214.1, 58.8), turned to 180 degrees
- moved J10 79.1 mm to (165.4, 45.0)
- moved C4 78.4 mm to (199.8, 85.8), turned to 270 degrees
- moved J11 73.8 mm to (113.3, 151.2)
- moved J4 73.7 mm to (121.4, 141.7)
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Connections:
- net SPI-5-Extra renamed Net-(J15-Pad1)
- C1 pad 1: +1V8 -> +3V3
- C5 pad 1: +1V8 -> +3V3
- C6 pad 1: +1V8 -> +3V3
- J15 pad 4: SPI-5-CS -> SPI_1_CS
- J15 pad 5: SPI-5-MISO -> SPI_1_MISO
- J15 pad 6: SPI-5-MOSI -> SPI_1_MOSI
- J15 pad 7: SPI-5-SCK -> SPI_1_SCK
- J15 pad 8: SPI-5-INT -> SPI_1_INT
- U1 pad 1: Net-(U1-Pad1) -> Steer5-Enc-Aout
- U1 pad 102: Drive2-PWMA -> Drive3-PWMA
- U1 pad 104: Net-(U1-Pad104) -> Drive2-Enc-Aout
- U1 pad 105: Drive3-INB2 -> Steer1-INB2
- U1 pad 109: Drive3-INB1 -> Steer1-INB1
- U1 pad 110: Net-(U1-Pad110) -> Steer1-INA2
- U1 pad 111: Net-(U1-Pad111) -> Steer1-Enc-Bout
- U1 pad 112: Net-(U1-Pad112) -> Steer1-Enc-Aout
- U1 pad 116: LED1 -> Net-(U1-Pad116)
- U1 pad 117: LED2 -> Steer2-INA1
- U1 pad 118: Net-(U1-Pad118) -> Steer2-INB2
- U1 pad 119: Net-(U1-Pad119) -> Steer2-INB1
- U1 pad 122: Net-(U1-Pad122) -> Steer2-INA2
- U1 pad 123: Net-(U1-Pad123) -> SPI_1_MOSI
- U1 pad 124: Steer2-Enc-Aout -> SPI_1_MISO
- U1 pad 125: Steer3-Enc-Bout -> SPI_1_CS
- U1 pad 126: Steer3-Enc-Aout -> SPI_1_SCK
- U1 pad 127: Net-(U1-Pad127) -> Steer6-Enc-Aout
- U1 pad 128: Net-(U1-Pad128) -> SPI_1_INT
- U1 pad 129: Net-(U1-Pad129) -> Drive4-Enc-Bout
- U1 pad 13: Drive2-B1 -> Drive3-INB1
- U1 pad 132: Steer1-INA1 -> Steer3-INA1
- U1 pad 137: CAN2-STBY -> Net-(U1-Pad137)
- U1 pad 141: Drive2-INA1 -> Drive3-INA1
- U1 pad 142: Steer1-INA2 -> Steer3-INA2
- U1 pad 15: Net-(U1-Pad15) -> Drive2-INA1
- U1 pad 17: Net-(U1-Pad17) -> (no net)
- U1 pad 18: SPI-5-CS -> Steer2-Enc-Bout
- U1 pad 19: SPI-5-SCK -> Steer2-Enc-Aout
- U1 pad 2: Net-(U1-Pad2) -> Steer3-INB2
- U1 pad 20: SPI-5-MISO -> Steer2-PWMA
- U1 pad 21: SPI-5-MOSI -> Steer2-PWMB
- U1 pad 22: Net-(U1-Pad22) -> Drive5-Enc-Bout
- U1 pad 24: Net-(U1-Pad24) -> Steer4-Enc-Bout
- U1 pad 3: Net-(U1-Pad3) -> Steer3-INB1
- U1 pad 34: Net-(U1-Pad34) -> Steer3-Enc-Bout
- U1 pad 35: Drive3-PWMB -> Steer1-PWMB
- U1 pad 36: Net-(U1-Pad36) -> Drive4-Enc-Aout
- U1 pad 4: Steer1-PWMA -> Steer3-PWMA
- U1 pad 40: Net-(U1-Pad40) -> Steer3-Enc-Aout
- U1 pad 41: Drive3-PWMA -> Steer1-PWMA
- U1 pad 43: Net-(U1-Pad43) -> Steer6-Enc-Bout
- U1 pad 44: Net-(U1-Pad44) -> Drive2-INA2
- U1 pad 46: Net-(U1-Pad46) -> Steer4-Enc-Aout
- U1 pad 47: Net-(U1-Pad47) -> Drive3-Enc-Bout
- U1 pad 48: CAN3-STBY -> CAN2-STBY
- U1 pad 49: Drive2-INA2 -> Drive3-INA2
- U1 pad 5: Steer1-PWMB -> Steer3-PWMB
- U1 pad 56: Drive1-Enc-Bout -> I2C-2-INT
- U1 pad 57: Drive1-Enc-Aout -> CAN1-STBY
- U1 pad 6: Net-(U1-Pad6) -> (no net)
- U1 pad 64: Drive2-B2 -> Drive3-INB2
- U1 pad 65: Net-(U1-Pad65) -> CAN3-STBY
- U1 pad 66: Net-(U1-Pad66) -> Drive2-B1
- U1 pad 67: Drive2-PWMB -> Drive3-PWMB
- U1 pad 68: Net-(U1-Pad68) -> Drive5-Enc-Aout
- U1 pad 69: Net-(U1-Pad69) -> Drive3-Enc-Aout
- U1 pad 7: Drive3-INA1 -> Steer1-INA1
- U1 pad 74: Net-(U1-Pad74) -> Drive2-B2
- U1 pad 77: Net-(U1-Pad77) -> Drive2-Enc-Bout
- U1 pad 78: Net-(U1-Pad78) -> I2C-2-EXTRA
- U1 pad 79: Net-(U1-Pad79) -> Drive6-Enc-Aout
- U1 pad 81: Steer2-PWMA -> Drive2-PWMA
- U1 pad 82: Steer2-PWMB -> Drive2-PWMB
- U1 pad 87: Drive2-Enc-Bout -> Net-(U1-Pad87)
- U1 pad 88: Drive2-Enc-Aout -> Steer5-Enc-Bout
- U1 pad 89: Drive3-Enc-Bout -> LED1
- U1 pad 90: Drive3-Enc-Aout -> LED2
- U1 pad 91: Steer1-Enc-Bout -> Net-(U1-Pad91)
- U1 pad 92: Steer1-Enc-Aout -> Net-(U1-Pad92)
- U1 pad 93: Steer2-Enc-Bout -> Drive6-Enc-Bout
- U1 pad 96: Net-(U1-Pad96) -> Drive1-Enc-Aout
- U1 pad 98: Net-(U1-Pad98) -> Drive1-Enc-Bout
- U1 pad GND: (no net) -> GND
- U3 pad 5: +1V8 -> +3V3
- U4 pad 5: +1V8 -> +3V3
- U5 pad 5: +1V8 -> +3V3
Routing:
- net Steer1-PWMA: track 12.1 -> 120.5 mm
- net GND: track 54.3 -> 150.3 mm, vias 10 -> 30
- net SPI_1_MOSI: track 0.00 -> 93.0 mm
- net CAN2-RXD: track 16.8 -> 86.2 mm
- net I2C-4-INT0: track 0.00 -> 69.2 mm
- net CAN3-RXD: track 0.00 -> 69.0 mm
- net +5V: track 25.1 -> 93.8 mm, vias 0 -> 18
- net SPI_1_MISO: track 0.00 -> 67.8 mm
- net CAN2-STBY: track 0.00 -> 64.5 mm
- net Net-(J20-Pad2): track 104.6 -> 43.0 mm
- net Net-(J17-Pad2): track 84.6 -> 23.0 mm
- net Steer2-PWMB: track 0.00 -> 60.0 mm
- net I2C-4-INT1: track 0.00 -> 59.1 mm
- net I2C-2-SCL: track 0.00 -> 54.9 mm
- net I2C-2-SDA: track 0.00 -> 52.6 mm
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- added copper zone on 5V, net +3V3
- added copper zone on 5V, net +5V
- added copper zone on GND, net GND
Other:
- board outline added: 184.5 x 118.4 mm
- board text added: "Drive 1"
- board text added: "Drive 2"
- board text added: "Drive 3"
- board text added: "I2C"
- board text added: "IMU"
- board text added: "SPI"
- board text added: "Steer 1 Enc"
- board text added: "Steer 2"
- board text added: "Steer 2 Enc"
- board text added: "Steer 3"
- board text added: "Steer 3 Enc"
- board text added: "Steer 4 Enc"
- board text added: "Steer 5 Enc"
- board text added: "Steer 6 Enc"
- board text added: "Steer1"
- board text removed: "DriverMotorEncoders"
- board text removed: "DrivingMotors"
- board text removed: "SteeringMotorEncoders"
- board text removed: "SteeringMotors"

Commit message: Add files via upload
Routing:
- net CAN3-RXD: track 69.0 -> 3.26 mm
- net GND: track 150.3 -> 138.1 mm, vias 30 -> 29
- net +3V3: track 44.6 -> 33.8 mm, vias 5 -> 3
- net +5V: track 93.8 -> 87.7 mm, vias 18 -> 17
- net CAN3-TXD: track 64.4 -> 65.2 mm, vias 0 -> 1
- net (no net): vias 1 -> 0
Other:
- board text added: "Drive 1 Enc"
- board text added: "Drive 2 Enc"
- board text added: "Drive 3 Enc"
- board text added: "Drive 4 Enc"
- board text added: "Drive 5 Enc"
- board text added: "Drive 6 Enc"

Commit message: Add files via upload
Parts:
- added J31: B3B-XH-A(LF)(SN), DriverBoard:JST3Way, F.Cu at (88.0, 47.9)
- added J32: B3B-XH-A(LF)(SN), DriverBoard:JST3Way, F.Cu at (88.0, 58.0)
- R1, R2: value CF14JT1K00 -> 1kΩ
Connections:
- U1 pad 139: Net-(U1-Pad139) -> TurretPWM1
- U1 pad 140: Net-(U1-Pad140) -> TurretPWM2
- U1 pad 6: (no net) -> Net-(U1-Pad6)
Routing:
- net +3V3: track 33.8 -> 129.4 mm, vias 3 -> 4
- net GND: track 138.1 -> 46.1 mm, vias 29 -> 8
- net +5V: track 87.7 -> 30.4 mm, vias 17 -> 3
- net TurretPWM1: track 0.00 -> 31.7 mm
- net TurretPWM2: track 0.00 -> 28.3 mm
- net CAN3-RXD: track 3.26 -> 0.00 mm
- net SabreTX: track 43.3 -> 41.9 mm
Other:
- board text added: "Turret Servo 1"
- board text added: "Turret Servo 2"
