File: RoboticsPCBS/DriverBoard/DriverBoard.sch (KiCad schematic (older format))
At the start: 41 parts, among them J1 B4B-XH-A(LF)(SN), J10 B8B-XH-ALFSN, J11 B8B-XH-ALFSN, J12 B8B-XH-ALFSN, J13 B8B-XH-ALFSN, J14 B6B-XH-ALFSN, J15 B8B-XH-ALFSN, J16 USB_B_Micro, J17 Conn_01x02_Male, J18 Conn_01x02_Male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

Commit message: Add files via upload
Parts:
- removed J16: USB_B_Micro, DriverBoard:MicroBVert, symbol Connector:USB_B_Micro
- removed J22: Conn_01x02_Male, DriverBoard:2PinHeader, symbol Connector:Conn_01x02_Male
- removed U1: STM32F767ZITx, DriverBoard:STM32, symbol MCU_ST_STM32F7:STM32F767ZITx
- removed U2: FT230XS, DriverBoard:FT230XS, symbol Interface_USB:FT230XS
- added J24, J25, J26, J27, J28, J29, J30: B4B-XH-A(LF)(SN), DriverBoard:JST4Way, symbol DriverBoard-rescue:B4B-XH-A(LF)(SN)-JST4Way
- added U1: STM32F767ZITx, DriverBoard:STM32, symbol stm32f767zitx_rev1:STM32F767ZITx
- J1, J2, J3, J4, J5, J6: symbol JST4Way:B4B-XH-A(LF)(SN) -> DriverBoard-rescue:B4B-XH-A(LF)(SN)-JST4Way
- J10, J11, J12, J13, J15, J8, J9: symbol JST8Way:B8B-XH-ALFSN -> DriverBoard-rescue:B8B-XH-ALFSN-JST8Way
- J14, J7: symbol JST6Way:B6B-XH-ALFSN -> DriverBoard-rescue:B6B-XH-ALFSN-JST6Way
- J19, J20, J21: symbol JST2Way:B2B-XH-A(LF)(SN) -> DriverBoard-rescue:B2B-XH-A(LF)(SN)-JST2Way
- R1, R2: footprint DriverBoard:LEDResistor -> DriverBoard:0603Footprint; symbol LEDResistor:CF14JT1K00 -> DriverBoard-rescue:CF14JT1K00-LEDResistor
- U3, U4, U5: symbol MCP2562:MCP2562-E_SN -> DriverBoard-rescue:MCP2562-E_SN-MCP2562
Connections:
- net +1V8 is gone; now on net +3V3: C1.1, C5.1, C6.1, U3.5 (VIO), U4.5 (VIO), U5.5 (VIO)
- net +3V3: now also U1.146 (3v3_1), U1.147 (3v3_2), U1.151 (3v3_3)
- net +5V: now also J24.4, J25.4, J26.4, J27.4, J28.4, J29.4, U1.148 (5V), U1.152 (5v_2)
- net CAN1-RXD: now also U1.114 (PD0)
- net CAN1-STBY: now also U1.57 (PG1)
- net CAN1-TXD: now also U1.115 (PD1)
- net CAN2-RXD: now also U1.135 (PB5)
- net CAN2-STBY: now also U1.48 (PB2)
- net CAN2-TXD: now also U1.136 (PB6)
- net CAN3-RXD: now also U1.133 (PB3)
- net CAN3-STBY: now also U1.65 (PE12)
- net CAN3-TXD: now also U1.134 (PB4)
- net Drive1-Enc-Aout: now also U1.96 (PC6)
- net Drive1-Enc-Bout: now also U1.98 (PC8)
- net Drive1-INA1: now also U1.75 (PB14)
- net Drive1-INA2: now also U1.76 (PB15)
- net Drive1-INB1: now also U1.70 (PB11)
- net Drive1-INB2: now also U1.97 (PC7)
- net Drive1-PWMA: now also U1.100 (PA8)
- net Drive1-PWMB: now also U1.101 (PA9)
- net Drive2-B1: now also U1.66 (PE13)
- net Drive2-B2: now also U1.74 (PB13)
- net Drive2-Enc-Aout: now also U1.104 (PA12)
- net Drive2-Enc-Bout: now also U1.77 (PD8)
- net Drive2-INA1: now also U1.15 (PF5)
- net Drive2-INA2: now also U1.44 (PC4)
- net Drive2-PWMA: now also U1.81 (PD12)
- net Drive2-PWMB: now also U1.82 (PD13)
- net Drive3-Enc-Aout: now also U1.69 (PB10)
- net Drive3-Enc-Bout: now also U1.47 (PB1)
- net Drive3-INA1: now also U1.141 (PE0)
- net Drive3-INA2: now also U1.49 (PF11)
- net Drive3-INB1: now also U1.13 (PF3)
- net Drive3-INB2: now also U1.64 (PE11)
- net Drive3-PWMA: now also U1.102 (PA10)
- net Drive3-PWMB: now also U1.67 (PE14)
- net GND: now also J24.3, J25.3, J26.3, J27.3, J28.3, J29.3
- net I2C-2-EXTRA: now also U1.12 (PF2), U1.78 (PD9)
- net I2C-2-INT: now also U1.56 (PG0)
- net I2C-2-SCL: now also U1.11 (PF1)
- net I2C-2-SDA: now also U1.10 (PF0)
- net I2C-4-INT0: now also U1.53 (PF13)
- net I2C-4-INT1: now also U1.50 (PF12)
- net I2C-4-SCL: now also U1.54 (PF14)
- net I2C-4-SDA: now also U1.55 (PF15)
- net LED1: now also U1.89 (PG4)
- net LED2: now also U1.90 (PG5)
- net ROSReset: now also U1.80 (PD11)
- net SabreTX: now also J30.1, J30.2, J30.3, J30.4, U1.113 (PC12)
- net Steer1-Enc-Aout: now also U1.112 (PC11)
- net Steer1-Enc-Bout: now also U1.111 (PC10)
- net Steer1-INA1: now also U1.7 (PC13)
- net Steer1-INA2: now also U1.110 (PA15)
- net Steer1-INB1: now also U1.109 (PA14)
- net Steer1-INB2: now also U1.105 (PA13)
- net Steer1-PWMA: now also U1.41 (PA5)
- net Steer1-PWMB: now also U1.35 (PA1)
- net Steer2-Enc-Aout: now also U1.19 (PF7)
- net Steer2-Enc-Bout: now also U1.18 (PF6)
- net Steer2-INA1: now also U1.117 (PD3)
- net Steer2-INA2: now also U1.122 (PD6)
- net Steer2-INB1: now also U1.119 (PD5)
- net Steer2-INB2: now also U1.118 (PD4)
- net Steer2-PWMA: now also U1.20 (PF8)
- net Steer2-PWMB: now also U1.21 (PF9)
- net Steer3-Enc-Aout: now also U1.40 (PA4)
- net Steer3-Enc-Bout: now also U1.34 (PA0)
- net Steer3-INA1: now also U1.132 (PG15)
- net Steer3-INA2: now also U1.142 (PE1)
- net Steer3-INB1: now also U1.3 (PE4)
- net Steer3-INB2: now also U1.2 (PE3)
- net Steer3-PWMA: now also U1.4 (PE5), U1.85 (PD14)
- net Steer3-PWMB: now also U1.5 (PE6), U1.86 (PD15)
- net UART-7-CTS: now also U1.63 (PE10)
- net UART-7-RTS: now also U1.60 (PE9)
- net UART-7-RXD: now also U1.58 (PE7)
- net UART-7-TXD: now also U1.59 (PE8)
- net SPI-5-CS renamed SPI_1_CS
- net SPI_1_CS: now also U1.125 (PG10)
- net SPI-5-Extra: no longer names the net of J15.1
- net SPI-5-INT renamed SPI_1_INT
- net SPI_1_INT: now also U1.128 (PG13)
- net SPI-5-MISO renamed SPI_1_MISO
- net SPI_1_MISO: now also U1.124 (PG9)
- net SPI-5-MOSI renamed SPI_1_MOSI
- net SPI_1_MOSI: now also U1.123 (PD7)
- net SPI-5-SCK renamed SPI_1_SCK
- net SPI_1_SCK: now also U1.126 (PG11)
- new net Drive4-Enc-Aout: J29.2, U1.36 (PA2)
- new net Drive4-Enc-Bout: J29.1, U1.129 (PG14)
- new net Drive5-Enc-Aout: J24.2, U1.68 (PE15)
- new net Drive5-Enc-Bout: J24.1, U1.22 (PF10)
- new net Drive6-Enc-Aout: J25.2, U1.79 (PD10)
- new net Drive6-Enc-Bout: J25.1, U1.93 (PG8)
- new net Steer4-Enc-Aout: J26.2, U1.46 (PB0)
- new net Steer4-Enc-Bout: J26.1, U1.24 (PH1)
- new net Steer5-Enc-Aout: J27.2, U1.1 (PE2)
- new net Steer5-Enc-Bout: J27.1, U1.88 (PG3)
- new net Steer6-Enc-Aout: J28.2, U1.127 (PG12)
- new net Steer6-Enc-Bout: J28.1, U1.43 (PA7)
- no-connect marks 12 -> 20
Other:
- note added: "PWM Pins\n"
- note added: "Turret Servos\n"
- note removed: "UART-USB Breakout"
- moved on the sheet: J14, J15, J7

Commit message: Add files via upload
Parts:
- added J31, J32: B3B-XH-A(LF)(SN), DriverBoard:JST3Way, symbol Connector_Generic:Conn_01x03
- C1, C2, C3, C4, C5, C6, R3, R4, R5: footprint DriverBoard:0603Footprint -> DriverBoard:Footprint_0603
- D1, D2: footprint DriverBoard:1812Footprint -> DriverBoard:LED_1812
- R1, R2: value CF14JT1K00 -> 1kΩ; footprint DriverBoard:0603Footprint -> DriverBoard:Footprint_0603; symbol DriverBoard-rescue:CF14JT1K00-LEDResistor -> Device:R
Connections:
- net labels added: TurretPWM1, TurretPWM2
- wire segments 145 -> 150
- no-connect marks 20 -> 18
Other:
- note removed: "PWM Pins\n"
- moved on the sheet: D1, D2, J7
