File: DriverBoardV2/DriverBoard.kicad_pcb (KiCad board)
At the start: 4 copper layers, 177.2 x 102 mm, 48 parts, among them J1 B4B-XH-A(LF)(SN), J10 B8B-XH-ALFSN, J11 B8B-XH-ALFSN, J12 B8B-XH-ALFSN, J13 B8B-XH-ALFSN, J14 B6B-XH-ALFSN, J15 B8B-XH-ALFSN, J17 Jumper, J18 Jumper, J19 B2B-XH-A(LF)(SN), J2 B4B-XH-A(LF)(SN), J20 B2B-XH-A(LF)(SN), J21 B2B-XH-A(LF)(SN), J23 Jumper, J24 B4B-XH-A(LF)(SN), J25 B4B-XH-A(LF)(SN), J26 B4B-XH-A(LF)(SN), J27 B4B-XH-A(LF)(SN), J28 B4B-XH-A(LF)(SN), J29 B4B-XH-A(LF)(SN), J3 B4B-XH-A(LF)(SN), J30 B4B-XH-A(LF)(SN), J31 B3B-XH-A(LF)(SN), J32 B3B-XH-A(LF)(SN), J4 B4B-XH-A(LF)(SN), J5 B4B-XH-A(LF)(SN), J6 B4B-XH-A(LF)(SN), J7 B6B-XH-ALFSN, J8 B8B-XH-ALFSN, J9 B8B-XH-ALFSN, U1 STM32F767ZITx, U3 MCP2562-E_SN, U4 MCP2562-E_SN, U5 MCP2562-E_SN

Commit message: Update DriverBoard-rescue.dcm, DriverBoard-rescue.lib, and 33 more files...
Parts:
- added R6: 1k, DriverBoard:Footprint_0603, F.Cu at (190.7, 136.0)
- added R7: 1k, DriverBoard:Footprint_0603, F.Cu at (194.8, 136.0)
- added R8: 1k, DriverBoard:Footprint_0603, F.Cu at (198.3, 62.7)
- added R9: 1k, DriverBoard:Footprint_0603, F.Cu at (199.0, 60.1)
- moved R1 62.9 mm to (227.1, 118.4)
- moved R2 62.9 mm to (227.1, 112.2)
- moved D1 62.9 mm to (219.1, 118.3)
- moved D2 62.9 mm to (219.1, 112.2)
- moved J8 17.7 mm to (131.0, 55.0), turned to 180 degrees
- moved J10 17.5 mm to (182.9, 55.0), turned to 180 degrees
- moved J9 17.4 mm to (156.8, 55.0), turned to 180 degrees
- moved J14 12.5 mm to (191.5, 142.0), turned to 0 degrees
- moved J7 12.5 mm to (191.5, 55.0), turned to 0 degrees
- moved J2 7.81 mm to (61.0, 132.2), turned to 270 degrees
- moved J26 7.81 mm to (71.0, 132.2), turned to 270 degrees
- moved J1 7.57 mm to (61.0, 87.5), turned to 270 degrees
- moved J24 7.57 mm to (71.0, 72.5), turned to 270 degrees
- moved J25 7.57 mm to (71.0, 57.5), turned to 270 degrees
- moved J27 7.57 mm to (71.0, 117.5), turned to 270 degrees
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Routing:
- net LED1: track 0.00 -> 64.2 mm, vias 0 -> 1
- net LED2: track 0.00 -> 62.6 mm, vias 0 -> 1
- net CAN3-STBY: track 0.00 -> 33.8 mm
- net Steer1-PWMA: track 0.00 -> 30.7 mm, vias 0 -> 1
- net Drive5-Enc-Bout: track 79.8 -> 100.7 mm
- net +5V: track 29.0 -> 43.9 mm, vias 1 -> 6
- net I2C-4-INT0: track 12.5 -> 23.7 mm, vias 1 -> 2
- net +3V3: track 27.5 -> 18.1 mm, vias 4 -> 3
- net Net-(J18-Pad1): track 33.1 -> 40.1 mm
- net Net-(J17-Pad1): track 30.8 -> 36.7 mm
- net Net-(J19-Pad2): track 32.6 -> 27.2 mm
- net Net-(J19-Pad1): track 29.3 -> 34.6 mm
- net Net-(J21-Pad2): track 36.1 -> 31.3 mm
- net Net-(J20-Pad2): track 33.6 -> 28.9 mm
- net TurretPWM2: track 27.3 -> 23.9 mm
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