File: DriverBoardV2/DriverBoard.sch (KiCad schematic (older format))
At the start: 47 parts, among them J1 B4B-XH-A(LF)(SN), J10 B8B-XH-ALFSN, J11 B8B-XH-ALFSN, J12 B8B-XH-ALFSN, J13 B8B-XH-ALFSN, J14 B6B-XH-ALFSN, J15 B8B-XH-ALFSN, J17 Jumper, J18 Jumper, J19 B2B-XH-A(LF)(SN), J2 B4B-XH-A(LF)(SN), J20 B2B-XH-A(LF)(SN), J21 B2B-XH-A(LF)(SN), J23 Jumper, J24 B4B-XH-A(LF)(SN), J25 B4B-XH-A(LF)(SN), J26 B4B-XH-A(LF)(SN), J27 B4B-XH-A(LF)(SN), J28 B4B-XH-A(LF)(SN), J29 B4B-XH-A(LF)(SN), J3 B4B-XH-A(LF)(SN), J30 B4B-XH-A(LF)(SN), J31 B3B-XH-A(LF)(SN), J32 B3B-XH-A(LF)(SN), J4 B4B-XH-A(LF)(SN), J5 B4B-XH-A(LF)(SN), J6 B4B-XH-A(LF)(SN), J7 B6B-XH-ALFSN, J8 B8B-XH-ALFSN, J9 B8B-XH-ALFSN, U1 STM32F767ZITx, U3 MCP2562-E_SN, U4 MCP2562-E_SN, U5 MCP2562-E_SN

Commit message: Update DriverBoard-rescue.dcm, DriverBoard-rescue.lib, and 33 more files...
Parts:
- added R6, R7, R8, R9: 1k, DriverBoard:Footprint_0603, symbol DriverBoardSymbols:R
Connections:
- net +5V: now also R6.1, R7.1, R8.1, R9.1
- net I2C-2-SCL: now also R7.2
- net I2C-2-SDA: now also R6.2
- net I2C-4-SCL: now also R9.2
- net I2C-4-SDA: now also R8.2
- net Steer1-PWMB: now also U1.137 (PB7); no longer U1.35 (PA1)
- no-connect marks 17 -> 16
Other:
- note added: "I2C Pullups\n"
- moved on the sheet: J14, J15, J7
