File: DriverBoardV3/DriverBoard.kicad_pcb (KiCad board)
At the start: 4 copper layers, 177.2 x 102 mm, 49 parts, among them J1 B4B-XH-A(LF)(SN), J10 B8B-XH-ALFSN, J11 B8B-XH-ALFSN, J12 B8B-XH-ALFSN, J13 B8B-XH-ALFSN, J14 B6B-XH-ALFSN, J15 B8B-XH-ALFSN, J17 Jumper, J18 Jumper, J19 B2B-XH-A(LF)(SN), J2 B4B-XH-A(LF)(SN), J20 B2B-XH-A(LF)(SN), J21 B2B-XH-A(LF)(SN), J23 Jumper, J24 B4B-XH-A(LF)(SN), J25 B4B-XH-A(LF)(SN), J26 B4B-XH-A(LF)(SN), J27 B4B-XH-A(LF)(SN), J28 B4B-XH-A(LF)(SN), J29 B4B-XH-A(LF)(SN), J3 B4B-XH-A(LF)(SN), J30 B4B-XH-A(LF)(SN), J31 B3B-XH-A(LF)(SN), J32 B3B-XH-A(LF)(SN), J4 B4B-XH-A(LF)(SN), J5 B4B-XH-A(LF)(SN), J6 B4B-XH-A(LF)(SN), J7 B6B-XH-ALFSN, J8 B8B-XH-ALFSN, J9 B8B-XH-ALFSN, U1 STM32F767ZITx

Commit message: Update DriverBoard-rescue.dcm, DriverBoard-rescue.lib, and 33 more files...
Parts:
- removed J10, J9: B8B-XH-ALFSN, DriverBoard:JST8Way
- added U3: MCP2562-E_SN, DriverBoard:MCP2562, F.Cu at (190.5, 112.2)
- added U4: MCP2562-E_SN, DriverBoard:MCP2562, F.Cu at (191.5, 98.8)
- added U5: MCP2562-E_SN, DriverBoard:MCP2562, F.Cu at (192.0, 84.2)
- J8: value B8B-XH-ALFSN -> B3B-XH-A(LF)(SN); footprint DriverBoard:JST8Way -> DriverBoard:JST3Way
- moved J25 162.8 mm to (210.5, 141.5), turned to 180 degrees
- moved J2 161.7 mm to (203.0, 55.0), turned to 0 degrees
- moved J24 142.3 mm to (195.5, 141.5), turned to 180 degrees
- moved J4 141.8 mm to (188.2, 55.0), turned to 0 degrees
- moved J29 122.1 mm to (180.5, 141.5), turned to 180 degrees
- moved J6 121.9 mm to (173.2, 55.0), turned to 0 degrees
- moved J13 111.3 mm to (70.8, 82.3), turned to 90 degrees
- moved J1 102.5 mm to (158.2, 55.0), turned to 0 degrees
- moved J28 102.2 mm to (165.5, 141.5), turned to 180 degrees
- moved J8 99.9 mm to (80.2, 141.0), turned to 0 degrees
- moved J14 98.8 mm to (92.8, 141.8)
- moved R6 93.3 mm to (97.4, 136.5)
- moved R7 93.3 mm to (101.6, 136.5)
- moved J3 84.1 mm to (143.2, 55.0), turned to 0 degrees
- moved J7 83.3 mm to (108.2, 55.8)
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Connections:
- net Net-(J17-Pad1) renamed /CAN2L
- net Net-(J18-Pad1) renamed /CAN3L
- net Net-(J19-Pad1) renamed /CAN1L
- net Net-(J19-Pad2) renamed /CAN1H
- net Net-(J20-Pad2) renamed /CAN2H
- net Net-(J21-Pad2) renamed /CAN3H
- net ROSReset renamed Net-(U1-Pad80)
- net UART-7-CTS renamed Net-(U1-Pad63)
- net UART-7-RTS renamed Net-(U1-Pad60)
- net UART-7-RXD renamed Net-(U1-Pad58)
- net UART-7-TXD renamed Net-(U1-Pad59)
- J14 pad 6: +5V -> I2CPWRTOGGLE
- J8 pad 2: GND -> Net-(J8-Pad2)
- J8 pad 3: Drive1-PWMB -> Net-(J8-Pad3)
- R6 pad 1: +5V -> +3V3
- R7 pad 1: +5V -> +3V3
- R8 pad 1: +5V -> +3V3
- R9 pad 1: +5V -> +3V3
- U1 pad 100: Drive1-PWMA -> Net-(U1-Pad100)
- U1 pad 101: Drive1-PWMB -> Net-(U1-Pad101)
- U1 pad 102: Drive3-PWMA -> Net-(U1-Pad102)
- U1 pad 13: Drive3-INB1 -> Net-(U1-Pad13)
- U1 pad 132: Steer3-INA1 -> Net-(U1-Pad132)
- U1 pad 15: Drive2-INA1 -> Net-(U1-Pad15)
- U1 pad 44: Drive2-INA2 -> Net-(U1-Pad44)
- U1 pad 49: Drive3-INA1 -> Net-(U1-Pad49)
- U1 pad 53: Drive3-INA2 -> Net-(U1-Pad53)
- U1 pad 64: Drive3-INB2 -> Net-(U1-Pad64)
- U1 pad 66: Drive2-B1 -> Net-(U1-Pad66)
- U1 pad 67: Drive3-PWMB -> Net-(U1-Pad67)
- U1 pad 70: Drive1-INB1 -> Net-(U1-Pad70)
- U1 pad 74: Drive2-B2 -> Net-(U1-Pad74)
- U1 pad 75: Drive1-INA1 -> Net-(U1-Pad75)
- U1 pad 76: Drive1-INA2 -> Net-(U1-Pad76)
- U1 pad 81: Drive2-PWMA -> Net-(U1-Pad81)
- U1 pad 82: Drive2-PWMB -> Net-(U1-Pad82)
- U1 pad 97: Drive1-INB2 -> Net-(U1-Pad97)
Routing:
- net GND: vias 3 -> 0
Other:
- board size 177.2 x 102 mm -> 162.4 x 102 mm
- board text removed: "Drive 1"
- board text removed: "Drive 2"
- board text removed: "Drive 3"

Commit message: Update CoopReport.docx, DriverBoard-cache.lib, and 18 more files...
Parts:
- C1, C2, C3, C4, C5, C6: footprint DriverBoard:0603Footprint -> DriverBoard:Footprint_0603
- D1, D2: footprint DriverBoard:1812Footprint -> Footprint:D_0805_2012Metric
- R1, R2: value 1kΩ -> 120Ω; footprint DriverBoard:0603Footprint -> Footprint:R_0805_2012Metric_Pad1.20x1.40mm_HandSolder
- R3: footprint DriverBoard:0603Footprint -> Footprint:R_0805_2012Metric_Pad1.20x1.40mm_HandSolder
- R4, R5: value 120Ω -> R_Small; footprint DriverBoard:0603Footprint -> Footprint:R_0603_1608Metric_Pad0.98x0.95mm_HandSolder
- R6, R7, R8, R9: value 1k -> R_Small; footprint DriverBoard:Footprint_0603 -> Footprint:R_0603_1608Metric_Pad0.98x0.95mm_HandSolder
- U3, U4, U5: footprint DriverBoard:MCP2562 -> MCP2562:MCP2562
- moved R4 121.2 mm to (99.6, 63.5), turned to 0 degrees
- moved R5 119.3 mm to (99.7, 65.5), turned to 0 degrees
- moved J2 116.0 mm to (122.8, 138.8)
- moved J4 97.6 mm to (138.2, 138.8)
- moved J14 87.1 mm to (115.0, 57.5)
- moved J6 86.0 mm to (153.8, 138.8)
- moved J25 84.0 mm to (212.5, 57.5), turned to 0 degrees
- moved J24 84.0 mm to (197.0, 57.5), turned to 0 degrees
- moved J29 84.0 mm to (181.5, 57.5), turned to 0 degrees
- moved J8 83.8 mm to (82.0, 57.2)
- moved J32 83.3 mm to (93.5, 138.8), turned to 0 degrees
- moved J31 83.0 mm to (80.8, 138.5), turned to 0 degrees
- moved R6 77.4 mm to (122.1, 63.1)
- moved R7 77.1 mm to (125.2, 63.1), turned to 0 degrees
- moved D1 50.8 mm to (217.6, 65.5)
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Connections:
- net CAN1-RXD renamed /CAN1-RXD
- net CAN1-STBY renamed /CAN1-STBY
- net CAN1-TXD renamed /CAN1-TX
- net CAN2-RXD renamed /CAN2-RXD
- net CAN2-TXD renamed /CAN2-TX
- net CAN3-RXD renamed /CAN3-RXD
- net CAN3-TXD renamed /CAN3-TX
- net I2CPWRTOGGLE renamed /I2C-2-INT2
- D1 pad 2: LED1 -> /LED1
- D2 pad 2: LED2 -> /LED2
- J14 pad 1: I2C-2-EXTRA -> +3V3
- J14 pad 2: I2C-2-INT -> GND
- J14 pad 3: I2C-2-SCL -> /I2C-2-SDA
- J14 pad 4: I2C-2-SDA -> /I2C-2-SCL
- J14 pad 5: GND -> /I2C-2-INT
- J15 pad 1: Net-(J15-Pad1) -> /SPI-1-INT
- J15 pad 2: +5V -> /SPI-1-SCK
- J15 pad 3: GND -> /SPI-1-MOSI
- J15 pad 4: SPI_1_CS -> /SPI-1-MISO
- J15 pad 5: SPI_1_MISO -> /SPI-1-CS
- J15 pad 6: SPI_1_MOSI -> GND
- J15 pad 7: SPI_1_SCK -> +3V3
- J15 pad 8: SPI_1_INT -> Net-(J15-Pad8)
- J17 pad 2: /CAN2L -> Net-(J17-Pad2)
- J18 pad 1: /CAN3L -> Net-(J18-Pad1)
- J23 pad 2: /CAN1L -> Net-(J23-Pad2)
- J30 pad 1: SabreTX -> /SabreTX
- J30 pad 2: SabreTX -> /SabreTX
- J30 pad 3: SabreTX -> /SabreTX
- J30 pad 4: SabreTX -> /SabreTX
- J31 pad 1: +5V -> /TurretPWM1
- J31 pad 3: TurretPWM1 -> +5V
- J32 pad 3: TurretPWM2 -> /TurretPWM2
- J7 pad 1: +3V3 -> /I2C-1-Extra
- J7 pad 2: GND -> /I2C-1-INT
- J7 pad 3: I2C-4-SDA -> /I2C-1-SCL
- J7 pad 4: I2C-4-SCL -> /I2C-1-SDA
- J7 pad 5: I2C-4-INT1 -> GND
- J7 pad 6: I2C-4-INT0 -> +3V3
- R1 pad 1: GND -> Net-(J23-Pad2)
- R1 pad 2: Net-(D1-Pad1) -> /CAN1H
- R2 pad 1: Net-(D2-Pad1) -> Net-(J17-Pad2)
- R2 pad 2: GND -> /CAN2H
- R3 pad 1: /CAN1L -> Net-(J18-Pad1)
- R3 pad 2: /CAN1H -> /CAN3H
- R4 pad 1: /CAN2L -> +3V3
- R4 pad 2: /CAN2H -> /I2C-1-SDA
- R5 pad 1: /CAN3L -> +3V3
- R5 pad 2: /CAN3H -> /I2C-1-SCL
- R6 pad 2: I2C-2-SDA -> /I2C-3-SDA
- R7 pad 2: I2C-2-SCL -> /I2C-3-SCL
- R8 pad 1: +3V3 -> Net-(D1-Pad1)
- R8 pad 2: I2C-4-SDA -> GND
- R9 pad 1: +3V3 -> Net-(D2-Pad1)
- R9 pad 2: I2C-4-SCL -> GND
- U1 pad 1: Steer5-Enc-Aout -> Net-(U1-Pad1)
- U1 pad 10: I2C-2-SDA -> Net-(U1-Pad10)
- U1 pad 104: Drive2-Enc-Aout -> Net-(U1-Pad104)
- U1 pad 105: Steer1-INB2 -> Net-(U1-Pad105)
- U1 pad 109: Steer1-INB1 -> Net-(U1-Pad109)
- U1 pad 11: I2C-2-SCL -> Net-(U1-Pad11)
- U1 pad 110: Steer1-INA2 -> Net-(U1-Pad110)
- U1 pad 111: Steer1-Enc-Bout -> /SabreTX
- U1 pad 112: Steer1-Enc-Aout -> Net-(U1-Pad112)
- U1 pad 113: SabreTX -> Net-(U1-Pad113)
- U1 pad 117: Steer2-INA1 -> Net-(U1-Pad117)
- U1 pad 118: Steer2-INB2 -> Net-(U1-Pad118)
- U1 pad 119: Steer2-INB1 -> Net-(U1-Pad119)
- U1 pad 12: I2C-2-EXTRA -> Net-(U1-Pad12)
- U1 pad 122: Steer2-INA2 -> Net-(U1-Pad122)
- U1 pad 123: SPI_1_MOSI -> /SPI-1-MISO
- U1 pad 124: SPI_1_MISO -> /SPI-1-MOSI
- U1 pad 125: SPI_1_CS -> /SPI-1-CS
- U1 pad 126: SPI_1_SCK -> /SPI-1-SCK
- U1 pad 127: Steer6-Enc-Aout -> Net-(U1-Pad127)
- U1 pad 128: SPI_1_INT -> /SPI-1-INT
- U1 pad 129: Drive4-Enc-Bout -> Net-(U1-Pad129)
- U1 pad 137: Steer1-PWMB -> Net-(U1-Pad137)
- U1 pad 139: TurretPWM1 -> /I2C-1-SCL
- U1 pad 140: TurretPWM2 -> /I2C-1-SDA
- U1 pad 141: I2C-4-INT0 -> Net-(U1-Pad141)
- U1 pad 142: Steer3-INA2 -> Net-(U1-Pad142)
- U1 pad 18: Steer2-Enc-Bout -> /TurretPWM1
- U1 pad 19: Steer2-Enc-Aout -> /TurretPWM2
- U1 pad 2: Steer3-INB2 -> Net-(U1-Pad2)
- U1 pad 20: Steer2-PWMA -> Net-(U1-Pad20)
- U1 pad 21: Steer2-PWMB -> Net-(U1-Pad21)
- U1 pad 22: Drive5-Enc-Bout -> Net-(U1-Pad22)
- U1 pad 24: Steer4-Enc-Bout -> Net-(U1-Pad24)
- U1 pad 3: Steer3-INB1 -> Net-(U1-Pad3)
- U1 pad 34: Steer3-Enc-Bout -> Net-(U1-Pad34)
- U1 pad 36: Drive4-Enc-Aout -> Net-(U1-Pad36)
- U1 pad 4: Steer3-PWMA -> Net-(U1-Pad4)
- U1 pad 40: Steer3-Enc-Aout -> Net-(U1-Pad40)
- U1 pad 41: Steer1-PWMA -> Net-(U1-Pad41)
- U1 pad 43: Steer6-Enc-Bout -> Net-(U1-Pad43)
- U1 pad 46: Steer4-Enc-Aout -> Net-(U1-Pad46)
- U1 pad 47: Drive3-Enc-Bout -> Net-(U1-Pad47)
- U1 pad 48: CAN2-STBY -> Net-(U1-Pad48)
- U1 pad 5: Steer3-PWMB -> Net-(U1-Pad5)
- U1 pad 50: I2C-4-INT1 -> Net-(U1-Pad50)
- U1 pad 54: I2C-4-SCL -> Net-(U1-Pad54)
- U1 pad 55: I2C-4-SDA -> Net-(U1-Pad55)
- U1 pad 56: I2C-2-INT -> Net-(U1-Pad56)
- U1 pad 65: CAN3-STBY -> Net-(U1-Pad65)
- U1 pad 68: Drive5-Enc-Aout -> Net-(U1-Pad68)
- U1 pad 69: Drive3-Enc-Aout -> /I2C-2-SCL
- U1 pad 7: Steer1-INA1 -> Net-(U1-Pad7)
- U1 pad 70: Net-(U1-Pad70) -> /I2C-2-SDA
- U1 pad 77: Drive2-Enc-Bout -> Net-(U1-Pad77)
- U1 pad 78: I2C-2-EXTRA -> Net-(U1-Pad78)
- U1 pad 79: Drive6-Enc-Aout -> Net-(U1-Pad79)
- U1 pad 85: Steer3-PWMA -> Net-(U1-Pad85)
- U1 pad 86: Steer3-PWMB -> Net-(U1-Pad86)
- U1 pad 88: Steer5-Enc-Bout -> Net-(U1-Pad88)
- U1 pad 89: LED1 -> Net-(U1-Pad89)
- U1 pad 90: LED2 -> Net-(U1-Pad90)
- U1 pad 93: Drive6-Enc-Bout -> Net-(U1-Pad93)
- U1 pad 96: Drive1-Enc-Aout -> Net-(U1-Pad96)
- U1 pad 98: Drive1-Enc-Bout -> Net-(U1-Pad98)
- U4 pad 8: CAN2-STBY -> /CAN2-STBY
- U5 pad 8: CAN3-STBY -> /CAN3-STBY
Routing:
- net /SPI-1-MISO: track 0.00 -> 54.9 mm
- net /SPI-1-CS: track 0.00 -> 47.5 mm
- net /TurretPWM1: track 0.00 -> 44.1 mm
- net /SPI-1-MOSI: track 0.00 -> 31.8 mm
- net /TurretPWM2: track 0.00 -> 29.0 mm
- net /SPI-1-INT: track 0.00 -> 27.7 mm
- net /I2C-2-SCL: track 0.00 -> 24.9 mm
- net /SPI-1-SCK: track 0.00 -> 24.1 mm
- net /CAN1-STBY: track 0.00 -> 23.0 mm
- net /I2C-1-SDA: track 0.00 -> 22.6 mm
- net /I2C-1-SCL: track 0.00 -> 22.1 mm
- net /CAN1H: track 0.00 -> 21.7 mm
- net /CAN1L: track 0.00 -> 19.9 mm
- net /CAN1-TX: track 0.00 -> 19.8 mm
- net /CAN1-RXD: track 0.00 -> 15.7 mm
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Other:
- net class Default: clearance 0.2 -> 0.25; trace_width 0.25 -> 0.4
- net class Small added: clearance 0.25, trace_width 0.25, via_dia 0.8, via_drill 0.4
- rule trace_clearance: 0.2 -> 0.25
- board text added: "RC Out"
- board text removed: "CAN 1"
- board text removed: "CAN1"
- board text removed: "CAN2"
- board text removed: "CAN3"
- board text removed: "Drive 1 Enc"
- board text removed: "Drive 2 Enc"
- board text removed: "Drive 3 Enc"
- board text removed: "Drive 4 Enc"
- board text removed: "Drive 5 Enc"
- board text removed: "Drive 6 Enc"
- board text removed: "I2C"
- board text removed: "IMU"
- board text removed: "SPI"
- board text removed: "SabreTX"
- board text removed: "Steer 1 Enc"
- board text removed: "Steer 2"
- board text removed: "Steer 2 Enc"
- board text removed: "Steer 3"
- board text removed: "Steer 3 Enc"
- board text removed: "Steer 4 Enc"
- board text removed: "Steer 5 Enc"
- board text removed: "Steer 6 Enc"
- board text removed: "Steer1"
- board text removed: "Turret Servo 1"
- board text removed: "Turret Servo 2"

Commit message: Update DriverBoard.kicad_pcb and DriverBoard.kicad_pcb-bak
Parts:
- moved R5 30.4 mm to (129.9, 62.3), turned to 180 degrees
- moved R7 26.0 mm to (99.2, 62.3)
- moved C3 15.3 mm to (188.5, 99.2), turned to 90 degrees
- moved C5 9.54 mm to (201.6, 103.4), turned to 270 degrees
- moved R2 9.21 mm to (222.6, 94.0), turned to 90 degrees
- moved J21 8.03 mm to (216.6, 80.8), turned to 270 degrees
- moved R3 5.15 mm to (222.6, 79.2), turned to 90 degrees
- moved J18 4.69 mm to (222.6, 83.1), turned to 0 degrees
- moved R4 4.06 mm to (103.5, 62.3), turned to 180 degrees
- moved J20 3.50 mm to (217.0, 95.5), turned to 270 degrees
- moved J17 3.37 mm to (222.6, 100.3), turned to 180 degrees
- moved R6 1.97 mm to (123.9, 62.3)
- moved D2 1.58 mm to (217.0, 70.0)
- moved R9 1.40 mm to (222.5, 70.0)
- moved R8 1.28 mm to (222.5, 65.0)
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Routing:
- net Steer2-PWMB: track 0.00 -> 78.0 mm
- net /CAN2-RXD: track 0.00 -> 74.0 mm
- net Steer2-INB2: track 0.00 -> 71.2 mm
- net Steer2-INB1: track 0.00 -> 67.9 mm
- net /CAN3-RXD: track 0.00 -> 65.0 mm
- net Steer1-INA1: track 0.00 -> 64.6 mm
- net Steer2-PWMA: track 0.00 -> 64.2 mm
- net Steer1-INA2: track 0.00 -> 61.3 mm
- net Steer1-INB1: track 0.00 -> 59.7 mm
- net Steer2-INA2: track 0.00 -> 58.1 mm
- net Steer1-INB2: track 0.00 -> 57.3 mm
- net /CAN3-TX: track 0.00 -> 56.7 mm
- net Steer3-PWMB: track 0.00 -> 56.0 mm
- net Steer2-INA1: track 0.00 -> 54.6 mm
- net Steer3-INB2: track 0.00 -> 54.3 mm
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
Commit message: Update DriverBoard.kicad_pcb, DriverBoard.kicad_pcb-bak, and 39 more files...
Parts:
- added J8: Conn_01x03, DriverBoard:PinHeader_1x03_P2.54mm_Vertical, F.Cu at (129.5, 56.0)
- R1, R2: value 120Ω -> 1kΩ; footprint Footprint:R_0805_2012Metric_Pad1.20x1.40mm_HandSolder -> DriverBoard:R_0603_1608Metric_Pad0.98x0.95mm_HandSolder
- R3: footprint Footprint:R_0805_2012Metric_Pad1.20x1.40mm_HandSolder -> DriverBoard:R_0805_2012Metric_Pad1.20x1.40mm_HandSolder
- R4, R5: value R_Small -> 120Ω; footprint Footprint:R_0603_1608Metric_Pad0.98x0.95mm_HandSolder -> DriverBoard:R_0805_2012Metric_Pad1.20x1.40mm_HandSolder
- R6, R7, R8, R9: value R_Small -> 1k; footprint Footprint:R_0603_1608Metric_Pad0.98x0.95mm_HandSolder -> DriverBoard:R_0603_1608Metric_Pad0.98x0.95mm_HandSolder
- moved R4 123.3 mm to (222.5, 94.2), turned to 90 degrees
- moved R8 121.1 mm to (101.4, 62.3), turned to 180 degrees
- moved R9 117.4 mm to (105.3, 62.3), turned to 180 degrees
- moved R5 94.1 mm to (222.5, 79.2), turned to 90 degrees
- moved R1 43.6 mm to (222.7, 65.0), turned to 180 degrees
- moved R3 29.5 mm to (222.5, 108.8)
- moved J13 25.8 mm to (74.0, 107.0)
- moved J12 24.4 mm to (74.0, 82.2)
- moved R2 24.1 mm to (222.7, 70.0), turned to 0 degrees
- moved R7 21.4 mm to (120.6, 62.3)
- moved C2 8.82 mm to (192.0, 106.8), turned to 180 degrees
- moved Ce 8.14 mm to (192.0, 91.8), turned to 180 degrees
- moved C4 7.74 mm to (192.0, 76.4), turned to 180 degrees
- moved J2 7.53 mm to (130.2, 139.4), turned to 180 degrees
- moved J26 7.53 mm to (176.8, 139.4), turned to 180 degrees
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- renumbered C3 to Ce
Connections:
- net /CAN1-RXD renamed CAN1-RXD
- net /CAN1-STBY renamed CAN1-STBY
- net /CAN1-TX renamed CAN1-TXD
- net /CAN2-RXD renamed CAN2-RXD
- net /CAN2-TX renamed CAN2-TXD
- net /CAN3-RXD renamed CAN3-RXD
- net /CAN3-TX renamed CAN3-TXD
- net /SPI-1-CS renamed SPI_1_CS
- net /SPI-1-INT renamed SPI_1_INT
- net /SPI-1-MISO renamed SPI_1_MISO
- net /SPI-1-MOSI renamed SPI_1_MOSI
- net /SPI-1-SCK renamed SPI_1_SCK
- net /SabreTX renamed SabreTX
- net /TurretPWM1 renamed TurretPWM1
- D1 pad 2: /LED1 -> LED1
- D2 pad 2: /LED2 -> LED2
- J12 pad 3: Steer2-PWMB -> Steer3-PWMB
- J12 pad 4: Steer2-INB2 -> Steer3-INB2
- J12 pad 5: Steer2-INB1 -> Steer3-INB1
- J12 pad 6: Steer2-PWMA -> Steer3-PWMA
- J12 pad 7: Steer2-INA2 -> Steer3-INA2
- J12 pad 8: Steer2-INA1 -> Steer3-INA1
- J13 pad 3: Steer3-PWMB -> Steer2-PWMB
- J13 pad 4: Steer3-INB2 -> Steer2-INB2
- J13 pad 5: Steer3-INB1 -> Steer2-INB1
- J13 pad 6: Steer3-PWMA -> Steer2-PWMA
- J13 pad 7: Steer3-INA2 -> Steer2-INA2
- J13 pad 8: Steer3-INA1 -> Steer2-INA1
- J14 pad 1: +3V3 -> I2C-2-EXTRA
- J14 pad 2: GND -> I2C-2-INT
- J14 pad 3: /I2C-2-SDA -> I2C-2-SCL
- J14 pad 4: /I2C-2-SCL -> I2C-2-SDA
- J14 pad 5: /I2C-2-INT -> GND
- J14 pad 6: /I2C-2-INT2 -> Net-(J14-Pad6)
- J15 pad 7: +3V3 -> +5V
- J17 pad 1: /CAN2L -> Net-(J17-Pad1)
- J17 pad 2: Net-(J17-Pad2) -> /CAN2L
- J2 pad 1: Steer1-Enc-Bout -> +5V
- J2 pad 2: Steer1-Enc-Aout -> GND
- J2 pad 3: GND -> Steer1-Enc-Aout
- J2 pad 4: +5V -> Steer1-Enc-Bout
- J23 pad 1: /CAN1L -> Net-(J23-Pad1)
- J23 pad 2: Net-(J23-Pad2) -> /CAN1L
- J26 pad 1: Steer4-Enc-Bout -> +5V
- J26 pad 2: Steer4-Enc-Aout -> GND
- J26 pad 3: GND -> Steer4-Enc-Aout
- J26 pad 4: +5V -> Steer4-Enc-Bout
- J27 pad 1: Steer5-Enc-Bout -> +5V
- J27 pad 2: Steer5-Enc-Aout -> GND
- J27 pad 3: GND -> Steer5-Enc-Aout
- J27 pad 4: +5V -> Steer5-Enc-Bout
- J28 pad 1: Steer6-Enc-Bout -> +5V
- J28 pad 2: Steer6-Enc-Aout -> GND
- J28 pad 3: GND -> Steer6-Enc-Aout
- J28 pad 4: +5V -> Steer6-Enc-Bout
- J32 pad 1: +5V -> TurretPWM2
- J32 pad 3: /TurretPWM2 -> +5V
- J4 pad 1: Steer2-Enc-Bout -> +5V
- J4 pad 2: Steer2-Enc-Aout -> GND
- J4 pad 3: GND -> Steer2-Enc-Aout
- J4 pad 4: +5V -> Steer2-Enc-Bout
- J6 pad 1: Steer3-Enc-Bout -> +5V
- J6 pad 2: Steer3-Enc-Aout -> GND
- J6 pad 3: GND -> Steer3-Enc-Aout
- J6 pad 4: +5V -> Steer3-Enc-Bout
- J7 pad 1: /I2C-1-Extra -> +3V3
- J7 pad 2: /I2C-1-INT -> GND
- J7 pad 3: /I2C-1-SCL -> I2C-4-SDA
- J7 pad 4: /I2C-1-SDA -> I2C-4-SCL
- J7 pad 5: GND -> I2C-4-INT1
- J7 pad 6: +3V3 -> I2C-4-INT0
- R1 pad 1: Net-(J23-Pad2) -> GND
- R1 pad 2: /CAN1H -> Net-(D1-Pad1)
- R2 pad 1: Net-(J17-Pad2) -> Net-(D2-Pad1)
- R2 pad 2: /CAN2H -> GND
- R3 pad 1: Net-(J18-Pad1) -> Net-(J23-Pad1)
- R3 pad 2: /CAN3H -> /CAN1H
- R4 pad 1: +3V3 -> Net-(J17-Pad1)
- R4 pad 2: /I2C-1-SDA -> /CAN2H
- R5 pad 1: +3V3 -> Net-(J18-Pad1)
- R5 pad 2: /I2C-1-SCL -> /CAN3H
- R6 pad 2: /I2C-3-SDA -> I2C-2-SDA
- R7 pad 2: /I2C-3-SCL -> I2C-2-SCL
- R8 pad 1: Net-(D1-Pad1) -> Net-(R8-Pad1)
- R8 pad 2: GND -> I2C-4-SDA
- R9 pad 1: Net-(D2-Pad1) -> Net-(R8-Pad1)
- R9 pad 2: GND -> I2C-4-SCL
- U1 pad 100: Net-(U1-Pad100) -> Drive1-Enc-Aout
- U1 pad 101: Net-(U1-Pad101) -> Drive1-Enc-Bout
- U1 pad 103: Net-(U1-Pad103) -> I2C-2-EXTRA
- U1 pad 104: Net-(U1-Pad104) -> I2C-2-INT
- U1 pad 105: Net-(U1-Pad105) -> Steer1-Enc-Bout
- U1 pad 109: Net-(U1-Pad109) -> Steer1-Enc-Aout
- U1 pad 11: Net-(U1-Pad11) -> Steer4-Enc-Aout
- U1 pad 110: Net-(U1-Pad110) -> Steer3-INB2
- U1 pad 112: Net-(U1-Pad112) -> Steer1-INB2
- U1 pad 113: Net-(U1-Pad113) -> Steer1-INB1
- U1 pad 116: Net-(U1-Pad116) -> Steer1-INA2
- U1 pad 127: Net-(U1-Pad127) -> Steer6-Enc-Bout
- U1 pad 13: Net-(U1-Pad13) -> Drive4-Enc-Bout
- U1 pad 137: Net-(U1-Pad137) -> Steer2-Enc-Bout
- U1 pad 139: /I2C-1-SCL -> I2C-4-SCL
- U1 pad 140: /I2C-1-SDA -> I2C-4-SDA
- U1 pad 141: Net-(U1-Pad141) -> Drive5-Enc-Bout
- U1 pad 142: Net-(U1-Pad142) -> Steer5-Enc-Aout
- U1 pad 15: Net-(U1-Pad15) -> Drive2-Enc-Aout
- U1 pad 19: /TurretPWM2 -> TurretPWM2
- U1 pad 2: Net-(U1-Pad2) -> Steer4-Enc-Bout
- U1 pad 28: Net-(U1-Pad28) -> Steer3-Enc-Bout
- U1 pad 29: Net-(U1-Pad29) -> Steer3-Enc-Aout
- U1 pad 41: Net-(U1-Pad41) -> Steer2-INA1
- U1 pad 42: Net-(U1-Pad42) -> Steer2-INA2
- U1 pad 44: Net-(U1-Pad44) -> Drive2-Enc-Bout
- U1 pad 46: Net-(U1-Pad46) -> CAN2-STBY
- U1 pad 50: Net-(U1-Pad50) -> Steer2-INB2
- U1 pad 54: Net-(U1-Pad54) -> Drive3-Enc-Aout
- U1 pad 55: Net-(U1-Pad55) -> Drive4-Enc-Aout
- U1 pad 56: Net-(U1-Pad56) -> Steer5-Enc-Bout
- U1 pad 58: Net-(U1-Pad58) -> Drive3-Enc-Bout
- U1 pad 60: Net-(U1-Pad60) -> Steer2-PWMB
- U1 pad 68: Net-(U1-Pad68) -> CAN3-STBY
- U1 pad 69: /I2C-2-SCL -> I2C-2-SCL
- U1 pad 7: Net-(U1-Pad7) -> Steer2-Enc-Aout
- U1 pad 70: /I2C-2-SDA -> I2C-2-SDA
- U1 pad 73: Net-(U1-Pad73) -> Steer3-INB1
- U1 pad 74: Net-(U1-Pad74) -> Steer3-PWMA
- U1 pad 76: Net-(U1-Pad76) -> Steer3-INA2
- U1 pad 78: Net-(U1-Pad78) -> Steer6-Enc-Aout
- U1 pad 85: Net-(U1-Pad85) -> Steer2-PWMA
- U1 pad 86: Net-(U1-Pad86) -> Steer2-INB1
- U1 pad 87: Net-(U1-Pad87) -> Steer1-INA1
- U1 pad 89: Net-(U1-Pad89) -> LED1
- U1 pad 90: Net-(U1-Pad90) -> Drive6-Enc-Bout
- U1 pad 91: Net-(U1-Pad91) -> Drive6-Enc-Aout
- U1 pad 92: Net-(U1-Pad92) -> LED2
- U1 pad 93: Net-(U1-Pad93) -> Drive5-Enc-Aout
- U1 pad 96: Net-(U1-Pad96) -> Steer3-INA1
- U1 pad 97: Net-(U1-Pad97) -> Steer3-PWMB
- U1 pad 98: Net-(U1-Pad98) -> Steer1-PWMB
- U1 pad 99: Net-(U1-Pad99) -> Steer1-PWMA
- U4 pad 8: /CAN2-STBY -> CAN2-STBY
- U5 pad 8: /CAN3-STBY -> CAN3-STBY
Routing:
- net +5V: track 17.3 -> 123.5 mm
- net Steer3-INA1: track 0.00 -> 43.4 mm
- net Net-(U1-Pad96): track 42.5 -> 0.00 mm
- net I2C-2-SCL: track 0.00 -> 30.8 mm
- net TurretPWM2: track 0.00 -> 30.6 mm
- net CAN2-STBY: track 0.00 -> 29.6 mm
- net /TurretPWM2: track 29.0 -> 0.00 mm
- net Net-(U1-Pad46): track 28.5 -> 0.00 mm
- net CAN3-STBY: track 0.00 -> 25.6 mm
- net I2C-4-SDA: track 0.00 -> 25.3 mm
- net /I2C-2-SCL: track 24.9 -> 0.00 mm
- net /CAN3-STBY: track 24.7 -> 0.00 mm
- net /I2C-1-SDA: track 22.6 -> 0.00 mm
- net /I2C-1-SCL: track 22.1 -> 0.00 mm
- net LED2: track 0.00 -> 20.7 mm
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- added copper zone on PWR, net +5V
- removed copper zone on 5V, net +3V3
- removed copper zone on 5V, net +5V
Other:
- board size 162.4 x 102 mm -> 160.8 x 93.5 mm
- board text added: "120Ω"
- board text added: "1kΩ"
- board text added: "3.3V"
- board text added: "5V"
- board text added: "65Ω"
- board text added: "CAN1"
- board text added: "CAN2"
- board text added: "CAN3"
- board text added: "Drive1ENC"
- board text added: "Drive2ENC"
- board text added: "Drive3ENC"
- board text added: "Drive4ENC"
- board text added: "Drive5ENC"
- board text added: "DriveENC6"
- board text added: "I2C Out"
- board text added: "IMU"
- board text added: "SPI"
- board text added: "SabreTX"
- board text added: "SteerDriver1"
- board text added: "SteerDriver2"
- board text added: "SteerDriver3"
- board text added: "SteerENC1"
- board text added: "SteerENC2"
- board text added: "SteerENC3"
- board text added: "SteerENC4"
- board text added: "SteerENC5"
- board text added: "SteerENC6"
- board text added: "Turret1"
- board text added: "Turret2"
