File: DriverBoardV3/DriverBoard.sch (KiCad schematic (older format))
At the start: 48 parts, among them J1 B4B-XH-A(LF)(SN), J11 B8B-XH-ALFSN, J12 B8B-XH-ALFSN, J13 B8B-XH-ALFSN, J14 B6B-XH-ALFSN, J15 B8B-XH-ALFSN, J17 Jumper, J18 Jumper, J19 B2B-XH-A(LF)(SN), J2 B4B-XH-A(LF)(SN), J20 B2B-XH-A(LF)(SN), J21 B2B-XH-A(LF)(SN), J23 Jumper, J24 B4B-XH-A(LF)(SN), J25 B4B-XH-A(LF)(SN), J26 B4B-XH-A(LF)(SN), J27 B4B-XH-A(LF)(SN), J28 B4B-XH-A(LF)(SN), J29 B4B-XH-A(LF)(SN), J3 B4B-XH-A(LF)(SN), J30 B4B-XH-A(LF)(SN), J31 B3B-XH-A(LF)(SN), J32 B3B-XH-A(LF)(SN), J4 B4B-XH-A(LF)(SN), J5 B4B-XH-A(LF)(SN), J6 B4B-XH-A(LF)(SN), J7 B6B-XH-ALFSN, U1 STM32F767ZITx, U3 MCP2562-E_SN, U4 MCP2562-E_SN, U5 MCP2562-E_SN

Commit message: Update DriverBoard-rescue.dcm, DriverBoard-rescue.lib, and 33 more files...
Parts:
- added J8: B3B-XH-A(LF)(SN), DriverBoard:JST3Way, symbol DriverBoardSymbols:JST_XH_3POS
- U3, U4, U5: footprint DriverBoard:MCP2562 -> MCP2562:MCP2562
Connections:
- net CAN1L: now reaches J19.1, J23.1, J23.2, R3.1, U3.6 (CANL)
- net CAN1H: now reaches J19.2, R3.2, U3.7 (CANH)
- net CAN2L: now reaches J17.1, J17.2, J20.1, R4.1, U4.6 (CANL)
- net CAN2H: now reaches J20.2, R4.2, U4.7 (CANH)
- net CAN3L: now reaches J18.1, J18.2, J21.1, R5.1, U5.6 (CANL)
- net CAN3H: now reaches J21.2, R5.2, U5.7 (CANH)
- no-connect marks 13 -> 52
Other:
- note added: "RC Out"
Changed lines of the file:
@@
 L power:+3V3 #PWR0145
 U 1 1 61B721FF
-P 750 2050
-F 0 "#PWR0145" H 750 1900 50  0001 C CNN
-F 1 "+3V3" H 765 2223 50  0000 C CNN
-F 2 "" H 750 2050 50  0001 C CNN
-F 3 "" H 750 2050 50  0001 C CNN
-	1    750  2050
+P 750 2200
+F 0 "#PWR0145" H 750 2050 50  0001 C CNN
+F 1 "+3V3" H 765 2373 50  0000 C CNN
+F 2 "" H 750 2200 50  0001 C CNN
+F 3 "" H 750 2200 50  0001 C CNN
+	1    750  2200
 	1    0    0    -1
 $EndComp
@@
 Wire Wire Line
 	1100 2200 750  2200
-Wire Wire Line
-	750  2200 750  2050
 Wire Notes Line style solid
 	500  1800 2450 1800
@@
 F 0 "U3" H 13200 2917 50  0000 C CNN
 F 1 "MCP2562-E_SN" H 13200 2826 50  0000 C CNN
-F 2 "DriverBoard:MCP2562" H 13200 2450 50  0001 L BNN
+F 2 "MCP2562:MCP2562" H 13200 2450 50  0001 L BNN
 F 3 "" H 13200 2450 50  0001 L BNN
 F 4 "Microchip" H 13200 2450 50  0001 L BNN "MANUFACTURER"
@@
 F 0 "U4" H 13250 4617 50  0000 C CNN
 F 1 "MCP2562-E_SN" H 13250 4526 50  0000 C CNN
-F 2 "DriverBoard:MCP2562" H 13250 4150 50  0001 L BNN
+F 2 "MCP2562:MCP2562" H 13250 4150 50  0001 L BNN
 F 3 "" H 13250 4150 50  0001 L BNN
 F 4 "Microchip" H 13250 4150 50  0001 L BNN "MANUFACTURER"
@@
 F 0 "U5" H 13300 6317 50  0000 C CNN
 F 1 "MCP2562-E_SN" H 13300 6226 50  0000 C CNN
-F 2 "DriverBoard:MCP2562" H 13300 5850 50  0001 L BNN
+F 2 "MCP2562:MCP2562" H 13300 5850 50  0001 L BNN
 F 3 "" H 13300 5850 50  0001 L BNN
 F 4 "Microchip" H 13300 5850 50  0001 L BNN "MANUFACTURER"
@@
 	1300 1200 1900 1200
 $Comp
-L power:+3.3V #PWR?
+L power:+3.3V #PWR0110
 U 1 1 6245F100
 P 3250 1400
-F 0 "#PWR?" H 3250 1250 50  0001 C CNN
+F 0 "#PWR0110" H 3250 1250 50  0001 C CNN
 F 1 "+3.3V" H 3265 1573 50  0000 C CNN
 F 2 "" H 3250 1400 50  0001 C CNN
@@
 $EndComp
 $Comp
-L power:+3.3V #PWR?
+L power:+3.3V #PWR0120
 U 1 1 6246033A
 P 4250 1400
-F 0 "#PWR?" H 4250 1250 50  0001 C CNN
+F 0 "#PWR0120" H 4250 1250 50  0001 C CNN
 F 1 "+3.3V" H 4265 1573 50  0000 C CNN
 F 2 "" H 4250 1400 50  0001 C CNN
@@
 	1    0    0    -1
 $EndComp
-NoConn ~ 7950 1800
 $Comp
 L power:GND #PWR0119
@@
 Wire Wire Line
 	850  2245 850  2300
+$Comp
+L DriverBoardSymbols:JST_XH_3POS J8
+U 1 1 62539FBC
+P 5455 5465
+F 0 "J8" H 5410 5235 50  0000 L CNN
+F 1 "B3B-XH-A(LF)(SN)" H 5085 5700 50  0000 L CNN
+F 2 "DriverBoard:JST3Way" H 5455 5465 50  0001 C CNN
+F 3 "~" H 5455 5465 50  0001 C CNN
+	1    5455 5465
+	-1   0    0    1
+$EndComp
+Text Notes 5065 5100 0    50   ~ 0
+RC Out
+NoConn ~ 10350 8100
+NoConn ~ 10350 8000
+NoConn ~ 10350 7900
+NoConn ~ 10350 7000
+NoConn ~ 10350 6000
+NoConn ~ 10350 5800
+NoConn ~ 10350 5600
+NoConn ~ 10350 5500
+NoConn ~ 10350 5400
+NoConn ~ 10350 5300
+NoConn ~ 10350 5200
+NoConn ~ 10350 5100
+NoConn ~ 10350 4900
+NoConn ~ 10350 4800
+NoConn ~ 10350 4700
+NoConn ~ 10350 4600
+NoConn ~ 10350 4500
+NoConn ~ 10350 2800
+NoConn ~ 10350 2700
+NoConn ~ 10350 2600
+NoConn ~ 10350 2500
+NoConn ~ 10350 2300
+NoConn ~ 10350 2000
+NoConn ~ 10350 1800
+NoConn ~ 7950 3600
+NoConn ~ 7950 4000
+NoConn ~ 7950 4100
+NoConn ~ 7950 4900
+NoConn ~ 7950 5400
+NoConn ~ 7950 5500
+NoConn ~ 7950 5600
+NoConn ~ 7950 6200
+NoConn ~ 7950 6400
+NoConn ~ 7950 7500
+NoConn ~ 7950 7600
+NoConn ~ 7950 7700
+NoConn ~ 7950 7800
+NoConn ~ 7950 7900
+NoConn ~ 7950 8100
+NoConn ~ 7950 8200
+Text Label 12100 5950 0    50   ~ 0
+CAN3H
+Text Label 12250 6450 0    50   ~ 0
+CAN3L
+Text Label 12150 4750 0    50   ~ 0
+CAN2L
+Text Label 12100 4250 0    50   ~ 0
+CAN2H
+Text Label 12100 2550 0    50   ~ 0
+CAN1H
+Text Label 12150 3050 0    50   ~ 0
+CAN1L
 $EndSCHEMATC

Commit message: Update CoopReport.docx, DriverBoard-cache.lib, and 18 more files...
Parts:
- removed C1, C2, C3, C4, C5, C6: 0.1µF, DriverBoard:Footprint_0603, symbol DriverBoardSymbols:C
- removed D1, D2: LED, DriverBoard:LED_1812, symbol DriverBoardSymbols:LED
- removed J1, J2, J24, J25, J26, J27, J28, J29, J3, J30, J4, J5, J6: B4B-XH-A(LF)(SN), DriverBoard:JST4Way, symbol DriverBoardSymbols:JST_XH_4POS
- removed J11, J12, J13, J15: B8B-XH-ALFSN, DriverBoard:JST8Way, symbol DriverBoardSymbols:JST_XH_8POS
- removed J14, J7: B6B-XH-ALFSN, DriverBoard:JST6Way, symbol DriverBoardSymbols:JST_XH_6POS
- removed J17, J18, J23: Jumper, DriverBoard:2PinHeader, symbol DriverBoardSymbols:Jumper
- removed J19, J20, J21: B2B-XH-A(LF)(SN), DriverBoard:JST2Way, symbol DriverBoardSymbols:JST_XH_2POS
- removed J31, J32, J8: B3B-XH-A(LF)(SN), DriverBoard:JST3Way, symbol DriverBoardSymbols:JST_XH_3POS
- removed R1, R2: 1kΩ, DriverBoard:Footprint_0603, symbol DriverBoardSymbols:R
- removed R3, R4, R5: 120Ω, DriverBoard:Footprint_0603, symbol DriverBoardSymbols:R
- removed R6, R7, R8, R9: 1k, DriverBoard:Footprint_0603, symbol DriverBoardSymbols:R
- removed U1: STM32F767ZITx, DriverBoard:STM32, symbol DriverBoardSymbols:STM32F7
- removed U3, U4, U5: MCP2562-E_SN, MCP2562:MCP2562, symbol DriverBoardSymbols:MCP2562
Connections:
- no-connect marks 52 -> 0
Other:
- note removed: "CAN Transcievers"
- note removed: "CS"
- note removed: "Driver Board"
- note removed: "Driver Motor Encoders\n"
- note removed: "Extra"
- note removed: "GND"
- note removed: "Hall Sensor A Vout"
- note removed: "Hall Sensor B Vout"
- note removed: "Hall Sensor GND"
- note removed: "Hall Sensor VCC"
- note removed: "I2C Connector"
- note removed: "I2C Pullups\n"
- note removed: "IMU"
- note removed: "INT"
- note removed: "MISO"
- note removed: "MOSI"
- note removed: "MotorDrivers (Steering Motors)\n"
- note removed: "Primary"
- note removed: "RC Out"
- note removed: "SCK\n"
- note removed: "SPI Connector"
- note removed: "SabreTooth TX"
- note removed: "Secondary"
- note removed: "Status LED's\n"
- note removed: "Steering Motor Encoders\n"
- note removed: "Tertiary"
- note removed: "Timer 4 Channel 1\n"
- note removed: "Timer 4 Channel 2\n\n\n\n"
- note removed: "Timer 4 Channel 3\n"
- note removed: "Timer 4 Channel 4\n"
- note removed: "Timer9 Channel 1"
- note removed: "Timer9 Channel 2\n"
- note removed: "Turret Servos\n"
- note removed: "VCC"

Commit message: Update DriverBoard.kicad_pcb, DriverBoard.kicad_pcb-bak, and 39 more files...
Parts:
- added C1: 0.1µF, DriverBoard:Footprint_0603, symbol DriverBoardSymbols:C
- added C2, C3, C4, C5, C6: 0.1µF, DriverBoard:C_0603_1608Metric_Pad1.08x0.95mm_HandSolder, symbol DriverBoardSymbols:C
- added D1, D2: LED, DriverBoard:LY R976-PS-36, symbol DriverBoardSymbols:LED
- added J1, J2, J24, J25, J26, J27, J28, J29, J3, J30, J4, J5, J6: B4B-XH-A(LF)(SN), DriverBoard:JST4Way, symbol DriverBoardSymbols:JST_XH_4POS
- added J11, J12, J13, J15: B8B-XH-ALFSN, DriverBoard:JST8Way, symbol DriverBoardSymbols:JST_XH_8POS
- added J14, J7: B6B-XH-ALFSN, DriverBoard:JST6Way, symbol DriverBoardSymbols:JST_XH_6POS
- added J17, J18, J23: Jumper, DriverBoard:2PinHeader, symbol DriverBoardSymbols:Jumper
- added J19, J20, J21: B2B-XH-A(LF)(SN), DriverBoard:JST2Way, symbol DriverBoardSymbols:JST_XH_2POS
- added J31, J32: B3B-XH-A(LF)(SN), DriverBoard:JST3Way, symbol DriverBoardSymbols:JST_XH_3POS
- added J8: Conn_01x03, DriverBoard:PinHeader_1x03_P2.54mm_Vertical, symbol DriverBoardSymbols:Conn_01x03
- added R1, R2: 1kΩ, DriverBoard:R_0603_1608Metric_Pad0.98x0.95mm_HandSolder, symbol DriverBoardSymbols:R
- added R3, R4, R5: 120Ω, DriverBoard:R_0805_2012Metric_Pad1.20x1.40mm_HandSolder, symbol DriverBoardSymbols:R
- added R6, R7, R8, R9: 1k, DriverBoard:R_0603_1608Metric_Pad0.98x0.95mm_HandSolder, symbol DriverBoardSymbols:R
- added U1: STM32F767ZITx, DriverBoard:STM32, symbol DriverBoardSymbols:STM32F7
- added U3, U4, U5: MCP2562-E_SN, DriverBoard:DIP787W45P254L1016H533Q8, symbol DriverBoardSymbols:MCP2562
Connections:
- new net: D1.1 (K), R1.2
- new net: D2.1 (K), R2.1
- new net: J14.6, J8.2 (Pin_2)
- new net: J23.1, R3.1
- new net: J17.1, R4.1
- new net: J18.1, R5.1
- new net: R8.1, R9.1
- new net +3V3: C1.1, C5.1, C6.1, J7.1, J8.3 (Pin_3), R6.1, R7.1, U1.146 (3v3_1), U1.147 (3v3_2), U1.151 (3v3_3), U3.5 (VIO), U4.5 (VIO), U5.5 (VIO)
- new net +5V: C2.1, C3.1, C4.1, J1.4, J15.7, J2.1, J24.4, J25.4, J26.1, J27.1, J28.1, J29.4, J3.4, J31.3 (Pin_3), J32.3 (Pin_3), J4.1, J5.4, J6.1, J8.1 (Pin_1), U1.148 (5V), U1.152 (5v_2), U3.3 (VDD), U4.3 (VDD), U5.3 (VDD)
- new net CAN1-RXD: U1.114 (PD0), U3.4 (RXD)
- new net CAN1-STBY: U1.57 (PG1), U3.8 (STBY)
- new net CAN1-TXD: U1.115 (PD1), U3.1 (TXD)
- new net CAN1H: J19.2, R3.2, U3.7 (CANH)
- new net CAN1L: J19.1, J23.2, U3.6 (CANL)
- new net CAN2-RXD: U1.135 (PB5), U4.4 (RXD)
- new net CAN2-STBY: U1.46 (PB0), U4.8 (STBY)
- new net CAN2-TXD: U1.136 (PB6), U4.1 (TXD)
- new net CAN2H: J20.2, R4.2, U4.7 (CANH)
- new net CAN2L: J17.2, J20.1, U4.6 (CANL)
- new net CAN3-RXD: U1.133 (PB3), U5.4 (RXD)
- new net CAN3-STBY: U1.68 (PE15), U5.8 (STBY)
- new net CAN3-TXD: U1.134 (PB4), U5.1 (TXD)
- new net CAN3H: J21.2, R5.2, U5.7 (CANH)
- new net CAN3L: J18.2, J21.1, U5.6 (CANL)
- new net Drive1-Enc-Aout: J1.2, U1.100 (PA8)
- new net Drive1-Enc-Bout: J1.1, U1.101 (PA9)
- new net Drive2-Enc-Aout: J3.2, U1.15 (PF5)
- new net Drive2-Enc-Bout: J3.1, U1.44 (PC4)
- new net Drive3-Enc-Aout: J5.2, U1.54 (PF14)
- new net Drive3-Enc-Bout: J5.1, U1.58 (PE7)
- new net Drive4-Enc-Aout: J29.2, U1.55 (PF15)
- new net Drive4-Enc-Bout: J29.1, U1.13 (PF3)
- new net Drive5-Enc-Aout: J24.2, U1.93 (PG8)
- new net Drive5-Enc-Bout: J24.1, U1.141 (PE0)
- new net Drive6-Enc-Aout: J25.2, U1.91 (PG6)
- new net Drive6-Enc-Bout: J25.1, U1.90 (PG5)
- new net GND: C1.2, C2.2, C3.2, C4.2, C5.2, C6.2, J1.3, J11.2, J12.2, J13.2, J14.5, J15.6, J2.2, J24.3, J25.3, J26.2, J27.2, J28.2, J29.3, J3.3, J31.2 (Pin_2), J32.2 (Pin_2), J4.2, J5.3, J6.2, J7.2, R1.1, R2.2, U1.158 (GND), U3.2 (VSS), U4.2 (VSS), U5.2 (VSS)
- new net I2C-2-EXTRA: J14.1, U1.103 (PA11)
- new net I2C-2-INT: J14.2, U1.104 (PA12)
- new net I2C-2-SCL: J14.3, R7.2, U1.69 (PB10)
- new net I2C-2-SDA: J14.4, R6.2, U1.70 (PB11)
- new net I2C-4-INT0: J7.6
- new net I2C-4-INT1: J7.5
- new net I2C-4-SCL: J7.4, R9.2, U1.139 (PB8)
- new net I2C-4-SDA: J7.3, R8.2, U1.140 (PB9)
- new net LED1: D1.2 (A), U1.89 (PG4)
- new net LED2: D2.2 (A), U1.92 (PG7)
- new net SPI_1_CS: J15.5, U1.125 (PG10)
- new net SPI_1_INT: J15.1, U1.128 (PG13)
- new net SPI_1_MISO: J15.4, U1.123 (PD7)
- new net SPI_1_MOSI: J15.3, U1.124 (PG9)
- new net SPI_1_SCK: J15.2, U1.126 (PG11)
- new net SabreTX: J30.1, J30.2, J30.3, J30.4, U1.111 (PC10)
- new net Steer1-Enc-Aout: J2.3, U1.109 (PA14)
- new net Steer1-Enc-Bout: J2.4, U1.105 (PA13)
- new net Steer1-INA1: J11.8, U1.87 (PG2)
- new net Steer1-INA2: J11.7, U1.116 (PD2)
- new net Steer1-INB1: J11.5, U1.113 (PC12)
- new net Steer1-INB2: J11.4, U1.112 (PC11)
- new net Steer1-PWMA: J11.6, U1.99 (PC9)
- new net Steer1-PWMB: J11.3, U1.98 (PC8)
- new net Steer2-Enc-Aout: J4.3, U1.7 (PC13)
- new net Steer2-Enc-Bout: J4.4, U1.137 (PB7)
- new net Steer2-INA1: J13.8, U1.41 (PA5)
- new net Steer2-INA2: J13.7, U1.42 (PA6)
- new net Steer2-INB1: J13.5, U1.86 (PD15)
- new net Steer2-INB2: J13.4, U1.50 (PF12)
- new net Steer2-PWMA: J13.6, U1.85 (PD14)
- new net Steer2-PWMB: J13.3, U1.60 (PE9)
- new net Steer3-Enc-Aout: J6.3, U1.29 (PC3)
- new net Steer3-Enc-Bout: J6.4, U1.28 (PC2)
- new net Steer3-INA1: J12.8, U1.96 (PC6)
- new net Steer3-INA2: J12.7, U1.76 (PB15)
- new net Steer3-INB1: J12.5, U1.73 (PB12)
- new net Steer3-INB2: J12.4, U1.110 (PA15)
- new net Steer3-PWMA: J12.6, U1.74 (PB13)
- new net Steer3-PWMB: J12.3, U1.97 (PC7)
- new net Steer4-Enc-Aout: J26.3, U1.11 (PF1)
- new net Steer4-Enc-Bout: J26.4, U1.2 (PE3)
- new net Steer5-Enc-Aout: J27.3, U1.142 (PE1)
- new net Steer5-Enc-Bout: J27.4, U1.56 (PG0)
- new net Steer6-Enc-Aout: J28.3, U1.78 (PD9)
- new net Steer6-Enc-Bout: J28.4, U1.127 (PG12)
- new net TurretPWM1: J31.1 (Pin_1), U1.18 (PF6)
- new net TurretPWM2: J32.1 (Pin_1), U1.19 (PF7)
- no-connect marks 0 -> 13
Other:
- note added: "CAN Transcievers"
- note added: "CS"
- note added: "Driver Motor Encoders\n"
- note added: "Extra"
- note added: "GND"
- note added: "Hall Sensor A Vout"
- note added: "Hall Sensor B Vout"
- note added: "Hall Sensor GND"
- note added: "Hall Sensor VCC"
- note added: "I2C Connector"
- note added: "I2C Pullups\n"
- note added: "IMU"
- note added: "INT"
- note added: "MISO"
- note added: "MOSI"
- note added: "MotorDrivers (Steering Motors)\n"
- note added: "PWR Selection\n"
- note added: "Primary"
- note added: "SCK\n"
- note added: "SPI Connector"
- note added: "SabreTooth TX"
- note added: "Secondary"
- note added: "Status LED's\n"
- note added: "Steering Motor Encoders\n"
- note added: "Tertiary"
- note added: "Turret Servos\n"
- note added: "VCC"
